File: Controllab.kicad_sch (KiCad schematic)
At the start: 56 parts, among them J3 TYPE-C-31-M-12, SW1 SW_Push, SW2 SW_Push, U2 ESP32-S3-MINI-1, U3 PN5321A3HN_C1xx, U4 AMS1117-3.3, Y1 Crystal

Commit message: La carte est prete
Parts:
- removed TP1_antenne1, TP2_antenne1: TestPoint, TestPoint:TestPoint_Pad_D1.0mm, symbol Connector:TestPoint
- added H1, H2, H3, H4: MountingHole, MountingHole:MountingHole_2.1mm, symbol Mechanical:MountingHole
- added J1: BM02B-GHS-TBT_LF__SN__N_, connecteur_pretty:JST_BM02B-GHS-TBT_LF__SN__N_, symbol BM02B-GHS-TBT_LF__SN__N_:BM02B-GHS-TBT_LF__SN__N_
- added JP5, JP6: SolderJumper_3_Open, Jumper:SolderJumper-3_P1.3mm_Open_Pad1.0x1.5mm, symbol Jumper:SolderJumper_3_Open
- R9: value 22K -> 2.7K
- SW1, SW2: footprint Button_Switch_SMD:SW_SPST_TL3342 -> Button_Switch_SMD:SW_SPST_PTS645Sx43SMTR92
Connections:
- net GND: now also J1.S1 (SHIELD), J1.S2 (SHIELD)
- net at C16.2, C18.1, R9.2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: no longer C17.2, C19.1, RQ2.1
- new net: ANT2.1 (T1), JP5.1 (A)
- new net: ANT2.2 (T2), JP6.1 (A)
- new net: JP5.2 (C), RQ1.2, TP2_TX2.1
- new net: J1.1, JP5.3 (B)
- new net: C17.2, C19.1, RQ2.1
- new net: JP6.2 (C), RQ2.2, TP1_TX1.1
- new net: J1.2, JP6.3 (B)
Other:
- moved on the sheet: ANT2, C16, C17, C18, C19, C20, L1, L2, R8, R9, RQ1, RQ2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

Commit message: ajout des noms sur la carte
Changed lines of the file:
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@@
-	)
-	(symbol
-		(lib_id "power:GND")
-		(at 241.3 125.73 0)
-		(unit 1)
-		(body_style 1)
-		(exclude_from_sim no)
-		(in_bom yes)
-		(on_board yes)
-		(in_pos_files yes)
-		(dnp no)
-		(fields_autoplaced yes)
-		(property "Reference" "#PWR033"
-			(at 241.3 132.08 0)
-			(hide yes)
-			(show_name no)
-			(do_not_autoplace no)
-			(effects
-				(font
-					(size 1.27 1.27)
-				)
-			)
-		)
-		(property "Value" "GND"
-			(at 241.3 130.81 0)
-			(show_name no)
-			(do_not_autoplace no)
-			(effects
-				(font
-					(size 1.27 1.27)
-				)
-			)
-		)
-		(property "Footprint" ""
-			(at 241.3 125.73 0)
-			(hide yes)
-			(show_name no)
-			(do_not_autoplace no)
-			(effects
-				(font
-					(size 1.27 1.27)
-				)
-			)
-		)
-		(property "Datasheet" ""
-			(at 241.3 125.73 0)
-			(hide yes)
-			(show_name no)
-			(do_not_autoplace no)
-			(effects
-				(font
-					(size 1.27 1.27)
-				)
-			)
-		)
-		(property "Description" "Power symbol creates a global label with name \"GND\" , ground"
-			(at 241.3 125.73 0)
-			(hide yes)
-			(show_name no)
-			(do_not_autoplace no)
-			(effects
-				(font
-					(size 1.27 1.27)
-				)
-			)
-		)
-		(pin "1"
-		)
-		(instances
-			(project "Controllab"
-				(path "/23877232-119e-43dd-a4d4-fa34d97aebd2"
-					(reference "#PWR033")
-					(unit 1)
-				)
-			)
-		)
 	)
 	(symbol
